File: PCB/GBARPi.sch (EAGLE design)
At the start: 55 parts, among them IC1 M68AW128MND, IC2 AD1895, U1 XC3S50ATQ144

Commit message: New CM4 version - untested
Parts:
- removed C1, C10, C11, C13, C14, C20, C21, C4, C5, C6, C7, C8: 2u2, rcl:C-EUC0805
- removed C12, C15, C16, C18, C19, C2, C22, C3, C9: 10u, rcl:C-EUC0805
- removed C17: (no value), rcl:C-EUC0805
- removed IC1: M68AW128MND, st-microelectronics:M68AW128MND
- removed IC2: AD1895, AD1895:AD1895
- removed PAD1, PAD2, PAD3, PAD4: (no value), wirepad:SMD2
- removed R1, R2, R3: (no value), rcl:R-EU_R0805
- removed SJ1, SJ2, SJ3, SJ4, SJ5, SJ6, SJ7: (no value), jumper:SJ
- removed TP1, TP10, TP11, TP2, TP3, TP4, TP5, TP6, TP7, TP8, TP9: TPTP10R, testpad:TPTP10R
- removed U$1, U$5: LD1117, LD1117:LD1117
- removed U$2: CONNECTOR, gameboy:CONNECTOR
- removed U$3: RPI-ZERO, RPI-Zero:RPI-ZERO
- removed U$4: ASE, crystal:ASE
- removed U1: XC3S50ATQ144, xilinx_spartan3_virtex4_and_5:XC3S50ATQ144
- added !BT_DISABLE, !EXTRST, !PI_LED_ACTIVITY, !PI_LED_PWR, !RPIBOOT, !WL_DISABLE, GLOBAL_EN, RUN_PG: TPB1,27, testpad:TPB1,27
- added BIAS-1.8V, JP1: (no value), q:SJS-NC3
- added BIAS-2.5V: (no value), q:SJ
- added CA301, CA302, CA303, CA304, CA305, CA306, CA307, CA308, CA309, CA401, CA402, CA403, CA404, CA405, CA406, CA407, CA606, CA607, CA608, CA701, CA702, CA703, CA704, CA705, CA706, CA901, CA902, CA903, CA904, CA905: (no value), rcl:C-EUC0402
- added CA601, CA604, CA605: (no value), rcl:C-EUC1206
- added CA602, CA603: (no value), rcl:C-EUC0603
- added CB601: 5.6uH, Wurth_Power Magnetics_WE-MAPI:WE-MAPI_4020_74438356056
- added CC501: 1043, c:1043
- added ENABLE_SEL: (no value), q:SJ2W
- added FC501: (no value), rcl:R-EU_R1206
- added KF1001, KF801: BSS138PW, q:BSS138PW
- added KF1002, QA801, QA802: NTS2101PT1G, q:NTS2101PT1G
- added KF401: ICE40UP5KSG48, c:ICE40UP5KSG48
- added KF901: STM32F042, c:STM32F042
- added PF_PI_ACTIVITY: (no value), led:LEDCHIP-LED0603
- added RA1001, RA1002, RA1003, RA102, RA301, RA701, RA801, RA802: 10k, rcl:R-EU_R0402
- added RA101: 1k, rcl:R-EU_R0402
- added RA302, RA309: 100, rcl:R-EU_R0402
- added RA303, RA304, RA305, RA306, RA307, RA308, RA401, RA601, RA602, RA603, RA604, RA605: (no value), rcl:R-EU_R0402
- added TA601: LT8336, c:LT8336
- added TA701: ADP322ACPZ-145-R7, c:ADP322ACPZ
- added X1: TC2050, q:TC2050
- added X2: TC2030, q:TC2030
- added XG101: CM4, c:CM4
- added XG201: GBA_CARTRIDGE_CONNECTOR, c:GBA_CARTRIDGE_CONNECTOR
Connections:
- removed net 3V3@2: U$3.3V3@2
- removed net AD1895_CLK: IC2.MCLK_IN, U1B0.IO_L12P_0VREF_0
- removed net DONE: TP9.TP, U1BVCCAUX.DONE
- removed net GBA_/CS1: U$2./RCS, U1B3.IO_L10N_3
- removed net GBA_/CS2: U$2./RS, U1B1.IO_L01P_1HDC
- removed net GBA_/RD: U$2./RD, U1B3.IO_L11P_3
- removed net GBA_/WR: U$2./WR, U1B3.IO_L10P_3
- removed net GBA_ON: R1.2, R2.1, U1B3.IO_L09P_3
- removed net I2S_CLK: IC2.SCLK_I, U$3.GPIO18
- removed net I2S_CLK_2: IC2.SCLK_O, U1B3.IO_L05N_3LHCLK1
- removed net I2S_DATA: IC2.SDATA_I, U$3.GPIO21
- removed net I2S_DATA_2: IC2.SDATA_O, U1B3.IO_L01N_3
- removed net I2S_LRCLK: IC2.LRCLK_I, U$3.GPIO19
- removed net I2S_LRCLK_2: IC2.LRCLK_O, U1B3.IO_L04N_3VREF_3
- removed net N$13: R3.2, U1B2.IO_L12P_2INIT_B
- removed net OSC: U$4.OUT, U1B3.IO_L08N_3LHCLK7
- removed net RAM_/CE: IC1G$1.!CE, U1B1.IO_L08N_1
- removed net RAM_/OE: IC1G$1.!OE, U1B0.IO_L10P_0
- removed net RAM_/WE: IC1G$1.!WE, U1B1.IO_L03N_1
- removed net RAM_ADDRESS0: IC1G$1.A0, U1B1.IO_L09P_1
- removed net RAM_ADDRESS1: IC1G$1.A1, U1B1.IO_L09N_1
- removed net RAM_ADDRESS10: IC1G$1.A10, U1B0.IO_L01N_0
- removed net RAM_ADDRESS11: IC1G$1.A11, U1B0.IO_L01P_0
- removed net RAM_ADDRESS12: IC1G$1.A12, U1B1.IO_L02N_1LDC0
- removed net RAM_ADDRESS13: IC1G$1.A13, U1B1.IO_L01N_1LDC2
- removed net RAM_ADDRESS14: IC1G$1.A14, U1B1.IO_1
- removed net RAM_ADDRESS15: IC1G$1.A15, U1B1.IO_L03P_1
- removed net RAM_ADDRESS16: IC1G$1.A16, U1B1.IO_L04P_1RHCLK0
- removed net RAM_ADDRESS2: IC1G$1.A2, U1B1.IO_L10P_1
- removed net RAM_ADDRESS3: IC1G$1.A3, U1B1.IO_L11P_1
- removed net RAM_ADDRESS4: IC1G$1.A4, U1B1.IO_L10N_1
- removed net RAM_ADDRESS5: IC1G$1.A5, U1B0.IO_L11N_0
- removed net RAM_ADDRESS6: IC1G$1.A6, U1B0.IO_L11P_0
- removed net RAM_ADDRESS7: IC1G$1.A7, U1B0.IO_L10N_0
- removed net RAM_ADDRESS8: IC1G$1.A8, U1B0.IO_L02N_0
- removed net RAM_ADDRESS9: IC1G$1.A9, U1B0.IO_L02P_0VREF_0
- removed net RAM_DATA0: IC1G$1.D0, U1B1.IO_L08P_1
- removed net RAM_DATA1: IC1G$1.D1, U1B1.IO_L07N_1RHCLK7
- removed net RAM_DATA10: IC1G$1.D10, U1B0.IO_L04N_0
- removed net RAM_DATA11: IC1G$1.D11, U1B0.IO_L03N_0
- removed net RAM_DATA12: IC1G$1.D12, U1B0.IO_L08P_0GCLK8
- removed net RAM_DATA13: IC1G$1.D13, U1B0.IO_L09P_0GCLK10
- removed net RAM_DATA14: IC1G$1.D14, U1B0.IO_L08N_0GCLK9
- removed net RAM_DATA15: IC1G$1.D15, U1B0.IO_L09N_0GCLK11
- removed net RAM_DATA2: IC1G$1.D2, U1B1.IO_L06N_1RHCLK5
- removed net RAM_DATA3: IC1G$1.D3, U1B1.IO_L07P_1IRDY1RHCLK6
- removed net RAM_DATA4: IC1G$1.D4, U1B1.IO_L06P_1RHCLK4
- removed net RAM_DATA5: IC1G$1.D5, U1B1.IO_L05N_1TRDY1RHCLK3
- removed net RAM_DATA6: IC1G$1.D6, U1B1.IO_L05P_1RHCLK2
- removed net RAM_DATA7: IC1G$1.D7, U1B1.IO_L04N_1RHCLK1
- removed net RAM_DATA8: IC1G$1.D8, U1B0.IO_L04P_0
- removed net RAM_DATA9: IC1G$1.D9, U1B0.IO_L03P_0
- removed net RPI_37: SJ7.1, U$3.GPIO26
- removed net RPI_PIN13: U$3.GPIO27/GEN2, U1B3.IO_L02N_3
- removed net RPI_PIN16: U$3.GEN4/GPIO23, U1B3.IO_L01P_3
- removed net RPI_PIN18: U$3.GEN5/GPIO24, U1B3.IO_L02P_3
- removed net RPI_PIN7: U$3.GPIO4/GCKL, U1B3.IO_L03N_3
- removed net RPI_RXD0: U$3.RXD0/GPIO15, U1B3.IO_L03P_3
- removed net RPI_TXD0: U$3.TXD0/GPIO14, U1B3.IO_L04P_3
- removed net SPI0_CS: U$3.!CE0!/GPIO8, U1B0.IP_0
- removed net SPI0_MISO: U$3.GPIO9/MISO
- removed net SPI0_MOSI: U$3.GPIO10/MOSI, U1B0.IO_0
- removed net SPI0_SCLK: U$3.GPIO11/SCLK, U1B3.IO_L05P_3LHCLK0
- removed net TCK: TP1.TP, U1BVCCAUX.TCK
- removed net TDI: TP4.TP, U1BVCCAUX.TDI
- removed net TDO: TP2.TP, U1BVCCAUX.TDO
- removed net TMS: TP3.TP, U1BVCCAUX.TMS
- removed net VCC: C1.1, C11.1, C12.1, C13.1, C14.1, C15.1, C18.1, C19.1, C2.1, C20.1, C21.1, C22.1, IC1P.VCC@1, IC1P.VCC@2, IC2.SMODE_IN_0, IC2.SMODE_OUT_0, IC2.VDD_CORE, IC2.VDD_IO, IC2.WLNGTH_OUT_0, IC2.WLNGTH_OUT_1, PAD1.P, PAD2.P, PAD3.P, PAD4.P, R3.1, SJ1.2, SJ3.1, SJ4.1, SJ5.1, SJ6.1, TP6.TP, U$1.VIN, U$4.TRI, U$4.VDD, U1B0.VCCO_00, U1B0.VCCO_01, U1B1.VCCO_10, U1B1.VCCO_11, U1B2.IO_L01N_2M0, U1B2.IO_L01P_2M1, U1B2.IO_L03N_2VS1, U1B2.IO_L04N_2VS0, U1B2.IO_L04P_2VS2, U1B2.VCCO_20, U1B2.VCCO_21, U1B3.VCCO_30, U1B3.VCCO_31, U1BVCCAUX.PROG_B, U1BVCCAUX.VCCAUX0, U1BVCCAUX.VCCAUX1, U1BVCCAUX.VCCAUX2, U1BVCCAUX.VCCAUX3
- removed net VCCINT: C10.1, C3.1, C4.1, C5.1, C6.1, C7.1, C8.1, C9.1, U$1.VOUT, U1BVCCINT.VCCINT0, U1BVCCINT.VCCINT1, U1BVCCINT.VCCINT2, U1BVCCINT.VCCINT3
- new net !BT_DISABLE: !BT_DISABLE.TP, XG101.!BT_DISABLE
- new net !EXTRST: !EXTRST.TP, XG101.!EXTRST
- new net !GBA_CS1: KF401.IOB_8A, XG201./RCS
- new net !GBA_CS2: KF901.PF1-OSC_OUT, XG201./RS
- new net !GBA_RD: KF401.IOB_9B, KF901.PB8, XG201./RD
- new net !GBA_WR: KF401.IOB_6A, KF901.PA10, XG201./WR
- new net !PI_LED_ACTIVITY: !PI_LED_ACTIVITY.TP, PF_PI_ACTIVITY.C, XG101.!PI_LED_ACTIVITY
- new net !PI_LED_PWR: !PI_LED_PWR.TP, XG101.!PI_LED_PWR
- new net !RPIBOOT: !RPIBOOT.TP, XG101.!RPIBOOT
- new net !STM_RESET: KF901.!RST, X2.3
- new net !WL_DISABLE: !WL_DISABLE.TP, XG101.!WL_DISABLE
- new net +5V_PI: QA801.D, QA802.D, RA101.1, XG101.+5V_IN_77, XG101.+5V_IN_79, XG101.+5V_IN_81, XG101.+5V_IN_83, XG101.+5V_IN_85, XG101.+5V_IN_87
- new net +5V_PI_EN: KF801.G, KF901.PA9, RA802.2
- new net BAT: CA601.1, CA701.1, CA702.1, CA703.1, CB601.1, ENABLE_SEL.3, FC501.2, KF1002.S, RA1001.2, TA601.VIN, TA701.VBIAS, TA701.VIN1/VIN2, TA701.VIN3
- new net BATT_VOLTAGE: KF901.PA7, RA1002.1, RA1003.2
- new net BAT_UNFUSED: CC501.P, FC501.1
- new net CM4_3.3V_OUT: RA102.2, XG101.CM4_3.3V_OUT_84, XG101.CM4_3.3V_OUT_86, XG101.GPIO_VREF
- new net DCDC_EN: KF1001.G, KF901.PA8, TA601.EN/UVLO
- new net DIFF_BIAS: CA309.1, RA301.2, RA303.2, RA305.2, RA307.2, RA309.2
- new net GLOBAL_EN: GLOBAL_EN.TP, XG101.GLOBAL_EN
- new net HDMI_CLK_ICE_N: CA301.1, KF401.IOT_44B, RA301.1, RA302.2
- new net HDMI_CLK_ICE_P: CA302.1, KF401.IOT_45A_G1, RA302.1
- new net HDMI_CLK_N: CA301.2, XG101.HDMI0_CLK_N
- new net HDMI_CLK_P: CA302.2, XG101.HDMI0_CLK_P
- new net HDMI_SCL: KF401.IOB_0A, XG101.HDMI0_SCL
- new net HDMI_SDA: KF401.IOB_2A, XG101.HDMI0_SDA
- new net HDMI_TX0_ICE_N: CA303.1, KF401.IOT_42B, RA303.1, RA304.2
- new net HDMI_TX0_ICE_P: CA304.1, KF401.IOT_43A, RA304.1
- new net HDMI_TX0_N: CA303.2, XG101.HDMI0_TX0_N
- new net HDMI_TX0_P: CA304.2, XG101.HDMI0_TX0_P
- new net HDMI_TX1_ICE_N: CA305.1, KF401.IOT_38B, RA305.1, RA306.2
- new net HDMI_TX1_ICE_P: CA306.1, KF401.IOT_39A, RA306.1
- new net HDMI_TX1_N: CA305.2, XG101.HDMI0_TX1_N
- new net HDMI_TX1_P: CA306.2, XG101.HDMI0_TX1_P
- new net HDMI_TX2_ICE_N: CA307.1, KF401.IOT_36B, RA307.1, RA308.2
- new net HDMI_TX2_ICE_P: CA308.1, KF401.IOT_37A, RA308.1
- new net HDMI_TX2_N: CA307.2, XG101.HDMI0_TX2_N
- new net HDMI_TX2_P: CA308.2, XG101.HDMI0_TX2_P
- new net ICE_CDONE: KF401.CDONE, X1.7
- new net ICE_CRESET_B: KF401.CRESET_B, X1.9
- new net ICE_SCK: KF401.IOB_34A_SPI_SCK, X1.4
- new net ICE_SI: KF401.IOB_33B_SPI_SI, X1.8
- new net ICE_SO: KF401.IOB_32A_SPI_SO, X1.6
- new net ICE_SS: KF401.IOB_35B_SPI_SS, X1.10
- new net ICE_VCC: BIAS-1.8V.1, CA403.1, CA404.1, CA706.1, KF401.VCC@30, KF401.VCC@5, RA401.2, TA701.EN1, TA701.VOUT3
- new net ICE_VCCIO: CA405.1, CA406.1, CA407.1, CA704.1, JP1.1, KF401.SPI_VCCIO1, KF401.VCCIO_0, KF401.VCCIO_2, TA701.EN2, TA701.VOUT1, X1.1
- new net ICE_VPP_2V5: BIAS-2.5V.1, CA402.1, CA705.1, KF401.VPP_2V5, TA701.VOUT2
- new net LT8336_BST: CA607.2, TA601.BST
- new net N$1: XG101.HDMI0_CEC
- new net N$11: BIAS-1.8V.2, BIAS-2.5V.2, RA309.1
- new net N$2: RA101.2, XG101.HDMI0_HOTPLUG
- new net N$3: CA608.2, RA601.1, RA602.2, TA601.FB
- new net N$4: CA607.1, CB601.2, TA601.SW
- new net N$7: KF801.D, QA801.G, QA802.G, RA801.1
- new net RUN_PG: RUN_PG.TP, XG101.RUN_PG
- new net STM_SWCLK: KF901.PA14, X2.4
- new net STM_SWDIO: KF901.PA13, X2.2
- new net USB_N: KF901.PA11, XG101.USB_N
- new net USB_P: KF901.PA12, XG101.USB_P
- new net VCCPLL: CA401.1, KF401.VCCPLL, RA401.1
- net +3V3: now also CA901.1, CA902.1, CA903.1, CA904.1, CA905.1, JP1.2, KF901.VDD, KF901.VDDA, KF901.VDDIO2, X2.1; no longer SJ4.2, U$3.3V3@1
- net +5V: now also CA602.1, CA603.1, CA604.1, CA605.1, CA608.1, QA801.S, QA802.S, RA601.2, RA801.2, TA601.VOUT; no longer SJ2.2, SJ5.2, U$3.5V0@1, U$3.5V0@2
- net GBA_ADDRESS_DATA0: now also KF401.IOB_13B, KF901.PA0, XG201.A0; no longer U$2.A0, U1B3.IO_L11N_3
- net GBA_ADDRESS_DATA1: now also KF401.IOB_16A, KF901.PA1, XG201.A1; no longer U$2.A1, U1B3.IO_L12P_3
- net GBA_ADDRESS_DATA10: now also KF401.IOT_41A, XG201.A10; no longer U$2.A10, U1B2.IO_L08P_2GCLK14
- net GBA_ADDRESS_DATA11: now also KF401.IOT_46B_G0, XG201.A11; no longer U$2.A11, U1B2.IO_L09P_2GCLK0
- net GBA_ADDRESS_DATA12: now also KF401.IOT_48B, XG201.A12; no longer U$2.A12, U1B2.IO_L10P_2GCLK2
- net GBA_ADDRESS_DATA13: now also KF401.IOT_50B, XG201.A13; no longer U$2.A13, U1B2.IO_L09N_2GCLK1
- net GBA_ADDRESS_DATA14: now also KF401.IOT_49A, XG201.A14; no longer U$2.A14, U1B2.IO_L10N_2GCLK3
- net GBA_ADDRESS_DATA15: now also KF401.IOT_51A, XG201.A15; no longer U$2.A15, U1B2.IO_2MOSICSI_B
- net GBA_ADDRESS_DATA16: now also KF901.PB0, XG201.D0; no longer U$2.D0, U1B2.IO_L11P_2AWAKE
- net GBA_ADDRESS_DATA17: now also KF901.PB1, XG201.D1; no longer U$2.D1, U1B2.IO_L11N_2DOUT
- net GBA_ADDRESS_DATA18: now also KF901.PB2, XG201.D2; no longer U$2.D2, U1B2.IO_L12N_2D3
- net GBA_ADDRESS_DATA19: now also KF901.PB3, XG201.D3; no longer U$2.D3, U1B2.IO_L13P_2D2
- net GBA_ADDRESS_DATA2: now also KF401.IOB_18A, KF901.PA2, XG201.A2; no longer U$2.A2, U1B3.IO_L12N_3
- net GBA_ADDRESS_DATA20: now also KF901.PB4, XG201.D4; no longer U$2.D4, U1B2.IO_L14P_2D1
- net GBA_ADDRESS_DATA21: now also KF901.PB5, XG201.D5; no longer U$2.D5, U1B2.IO_L13N_2D0DINMISO
- net GBA_ADDRESS_DATA22: now also KF901.PB6, XG201.D6; no longer U$2.D6, U1B2.IO_L14N_2CCLK
- net GBA_ADDRESS_DATA23: now also KF901.PB7, XG201.D7; no longer U$2.D7, U1B1.IO_L02P_1LDC1
- net GBA_ADDRESS_DATA3: now also KF401.IOB_20A, KF901.PA3, XG201.A3; no longer U$2.A3, U1B2.IO_L02N_2CSO_B
- net GBA_ADDRESS_DATA4: now also KF401.IOB_22A, KF901.PA4, XG201.A4; no longer U$2.A4, U1B2.IO_L05P_2
- net GBA_ADDRESS_DATA5: now also KF401.IOB_24A, KF901.PA5, XG201.A5; no longer U$2.A5, U1B2.IO_L06P_2
- net GBA_ADDRESS_DATA6: now also KF401.IOB_31B, KF901.PA6, XG201.A6; no longer U$2.A6, U1B2.IO_L05N_2D7
- net GBA_ADDRESS_DATA7: now also KF401.IOB_29B, XG201.A7; no longer U$2.A7, U1B2.IO_L06N_2D6
- net GBA_ADDRESS_DATA8: now also KF401.IOB_25B_G3, XG201.A8; no longer U$2.A8, U1B2.IO_L07P_2D5
- net GBA_ADDRESS_DATA9: now also KF401.IOB_23B, XG201.A9; no longer U$2.A9, U1B2.IO_L07N_2D4
- net GBA_CLK: now also KF401.IOB_3B_G6, KF901.PF0-OSC_IN, XG201.NC; no longer TP8.TP, U$2.NC, U1B3.IO_L09N_3
- net GBA_IRQ: now also KF901.PA15, XG201.VIN; no longer TP11.TP, U$2.VIN
- net GBA_VCC: now also ENABLE_SEL.1, XG201.VDD; no longer R1.1, SJ1.1, U$2.VDD
- net GND: now also CA309.2, CA401.2, CA402.2, CA403.2, CA404.2, CA405.2, CA406.2, CA407.2, CA601.2, CA602.2, CA603.2, CA604.2, CA605.2, CA606.2, CA701.2, CA702.2, CA703.2, CA704.2, CA705.2, CA706.2, CA901.2, CA902.2, CA903.2, CA904.2, CA905.2, CC501.N, KF1001.S, KF401.GND, KF801.S, KF901.PF11-BOOT0, KF901.VSS, RA1003.1, RA602.1, RA603.1, RA605.1, RA802.1, TA601.GND, TA701.GND, X1.3, X2.5, XG101.GND1, XG101.GND107, XG101.GND108, XG101.GND113, XG101.GND114, XG101.GND119, XG101.GND120, XG101.GND125, XG101.GND126, XG101.GND13, XG101.GND131, XG101.GND132, XG101.GND137, XG101.GND138, XG101.GND14, XG101.GND144, XG101.GND150, XG101.GND155, XG101.GND156, XG101.GND161, XG101.GND162, XG101.GND167, XG101.GND168, XG101.GND173, XG101.GND174, XG101.GND179, XG101.GND180, XG101.GND185, XG101.GND186, XG101.GND191, XG101.GND192, XG101.GND197, XG101.GND198, XG101.GND2, XG101.GND22, XG101.GND23, XG101.GND32, XG101.GND33, XG101.GND42, XG101.GND43, XG101.GND52, XG101.GND53, XG101.GND59, XG101.GND60, XG101.GND65, XG101.GND66, XG101.GND7, XG101.GND71, XG101.GND74, XG101.GND8, XG101.GND98, XG201.GND; no longer C1.2, C10.2, C11.2, C12.2, C13.2, C14.2, C15.2, C16.2, C17.2, C18.2, C19.2, C2.2, C20.2, C21.2, C22.2, C3.2, C4.2, C5.2, C6.2, C7.2, C8.2, C9.2, IC1G$1.!LB, IC1G$1.!UB, IC1P.VSS@1, IC1P.VSS@2, IC2.BYPASS, IC2.DGND_21, IC2.DGND_8, IC2.MMODE_0, IC2.MMODE_1, IC2.MMODE_2, IC2.SMODE_IN_1, IC2.SMODE_IN_2, IC2.SMODE_OUT_1, IC2.TDM_IN, R2.2, TP5.TP, U$1.GND, U$2.GND, U$3.GND@1, U$3.GND@2, U$3.GND@3, U$3.GND@4, U$3.GND@6, U$3.GND@7, U$3.GND@8, U$4.GND, U$5.GND, U1B0.IO_L12N_0PUDC_B, U1B0.IP_0VREF_0, U1B1.IP_1VREF_10, U1B1.IP_1VREF_11, U1B1.SUSPEND, U1B2.IO_L02P_2M2, U1B3.IP_L13N_3VREF_3, U1B3.IP_L13P_3, U1BGND.GND0, U1BGND.GND1, U1BGND.GND10, U1BGND.GND11, U1BGND.GND12, U1BGND.GND2, U1BGND.GND3, U1BGND.GND4, U1BGND.GND5, U1BGND.GND6, U1BGND.GND7, U1BGND.GND8, U1BGND.GND9
- net N$10: now also ENABLE_SEL.2, RA701.1; no longer IC2.MUTE_IN, IC2.MUTE_OUT
- net N$12: now also PF_PI_ACTIVITY.A, RA102.1; no longer U1B0.IO_L06P_0GCLK4, U1B0.IO_L07P_0GCLK6
- net N$14: now also KF1001.D, KF1002.G, RA1001.1; no longer U1B0.IO_L06N_0GCLK5, U1B0.IO_L07N_0GCLK7
- net N$15: now also KF1002.D, RA1002.2; no longer IC2./RESET, SJ6.2, SJ7.2
- net N$5: now also RA603.2, TA601.RT; no longer SJ3.2, U$5.VOUT
- net N$6: now also RA604.1, RA605.2, TA601.SYNC/MODE; no longer TP7.TP, U1B3.IO_L08P_3TRDY2LHCLK6
- net N$8: now also CA606.1, RA604.2, TA601.INTVCC; no longer C16.1, C17.1, SJ2.1, U$5.VIN
- net N$9: now also RA701.2, TA701.EN3; no longer TP10.TP, U1B2.IO_L03P_2RDWR_B
Other:
- note added: "1.2 V"
- note added: "2.5 V"
- note added: "3.3 V"
- note added: "HDMI: - AC coupling - Bias - 100 Ohm Termination"
- note added: "Zone 1"
- note added: "Zone 10 Battery voltage measurement"
- note added: "Zone 2"
- note added: "Zone 3"
- note added: "Zone 4"
- note added: "Zone 5"
- note added: "Zone 6"
- note added: "Zone 7"
- note added: "Zone 8"
- note added: "Zone 9"
- note removed: "AD1895"
- note removed: "DRAM"
- note removed: "FPGA"
- note removed: "Oscillator"
- note removed: "Power"
- note removed: "Raspberry Pi Zero"
